Commit message: Initial commit

File: src/sam_bot_nav2_gz/src/description/sam_bot_description.urdf (robot description, URDF)
Before this commit: robot sam_bot, 7 links, 6 joints
Links:
- added link dirt_tank_link; collision box size=0.25 0.25 0.1; visual box size=0.25 0.25 0.1
- added link hard_brush_link; collision cylinder length=0.02 radius=0.05; visual cylinder length=0.02 radius=0.05
- added link soft_brush_link; collision cylinder length=0.02 radius=0.05; visual cylinder length=0.02 radius=0.05
Joints:
- added joint dirt_tank_joint: type fixed, parent base_link, child dirt_tank_link, origin xyz=-0.05 0 ${base_height/2}
- added joint hard_brush_joint: type continuous, parent base_link, child hard_brush_link, origin xyz=${base_length/2 - 0.02} ${-(base_width/2 - 0.06)} ${-(wheel_radius+wheel_zoff) - 0.005} rpy=0 0 0, axis 0 0 1
- added joint soft_brush_joint: type continuous, parent base_link, child soft_brush_link, origin xyz=${base_length/2 - 0.02} ${base_width/2 - 0.06} ${-(wheel_radius+wheel_zoff) - 0.005} rpy=0 0 0, axis 0 0 1
